Commit message: Change urdf package.

File: mobile_manipulator_assets/diablo_swingarm/description/urdf/diablo/diablo.xacro (robot description, xacro)
@@ -2,50 +2,50 @@
 <robot xmlns:xacro="http://ros.org/wiki/xacro" name="diablo">
     <!-- Include predefined materials -->
-    <xacro:include filename="$(find upright_asset)/description/urdf/common/materials.xacro"/>
-    <xacro:include filename="$(find upright_asset)/description/urdf/common/common.xacro"/>
+    <xacro:include filename="$(find robot_common)/include/robot_common/utilities/urdf/common.xacro"/>
+    <xacro:include filename="$(find robot_common)/include/robot_common/utilities/urdf/materials.xacro"/>
     <!-- Base Link -->
     <xacro:create_link name="diablo_base_link" mass="11.639" ixx="0.071628" ixy="-5.9879E-09" ixz="-0.00097471"
                        iyy="0.16274" iyz="-1.6369E-08" izz="0.14673"
-                       mesh_file="package://upright_asset/description/meshes/diablo/base_link.STL"
+                       mesh_file="package://diablo_swingarm/description/meshes/diablo/base_link.STL"
                        material_name="grey"/>
     <xacro:create_link name="left_motor" mass="1.3837" ixx="0.003352" ixy="2.7785E-09" ixz="-6.5913E-05" iyy="0.0034908"
                        iyz="4.5045E-10" izz="0.0034856"
-                       mesh_file="package://upright_asset/description/meshes/diablo/left_motor.STL"
+                       mesh_file="package://diablo_swingarm/description/meshes/diablo/left_motor.STL"
                        material_name="silver"/>
     <xacro:create_link name="left_leg1" mass="0.10382" ixx="3.6972E-05" ixy="2.4106E-05" ixz="4.3699E-10"
                        iyy="0.00029278" iyz="-4.1243E-11" izz="0.00032532"
-                       mesh_file="package://upright_asset/description/meshes/diablo/left_leg1.STL"
+                       mesh_file="package://diablo_swingarm/description/meshes/diablo/left_leg1.STL"
                        material_name="silver"/>
     <xacro:create_link name="left_leg2" mass="0.18218" ixx="4.1372E-05" ixy="5.1445E-09" ixz="-7.3659E-06"
                        iyy="0.00048219" iyz="2.5521E-11" izz="0.00050441"
-                       mesh_file="package://upright_asset/description/meshes/diablo/left_leg2.STL"
+                       mesh_file="package://diablo_swingarm/description/meshes/diablo/left_leg2.STL"
                        material_name="silver"/>
     <xacro:create_link name="left_wheel" mass="2.9494" ixx="0.0069338" ixy="2.8693E-09" ixz="4.6779E-09" iyy="0.006934"
                        iyz="-5.0441E-11" izz="0.012567"
-                       mesh_file="package://upright_asset/description/meshes/diablo/left_wheel.STL"
+                       mesh_file="package://diablo_swingarm/description/meshes/diablo/left_wheel.STL"
                        material_name="black"/>
     <xacro:create_link name="left_leg3" mass="0.071103" ixx="1.6657E-05" ixy="-5.5246E-06" ixz="3.9598E-14"
                        iyy="0.00017966" iyz="-6.5493E-15" izz="0.00019328"
-                       mesh_file="package://upright_asset/description/meshes/diablo/left_leg3.STL"
+                       mesh_file="package://diablo_swingarm/description/meshes/diablo/left_leg3.STL"
                        material_name="brown"/>
     <xacro:create_link name="right_motor" mass="1.3838" ixx="0.003352" ixy="-2.6527E-09" ixz="6.5914E-05"
                        iyy="0.0034908" iyz="-7.2968E-10" izz="0.0034856"
-                       mesh_file="package://upright_asset/description/meshes/diablo/right_motor.STL"
+                       mesh_file="package://diablo_swingarm/description/meshes/diablo/right_motor.STL"
                        material_name="silver"/>
     <xacro:create_link name="right_leg1" mass="0.10382" ixx="3.6972E-05" ixy="2.4106E-05" ixz="-4.3686E-10"
                        iyy="0.00029278" iyz="4.1459E-11" izz="0.00032532"
-                       mesh_file="package://upright_asset/description/meshes/diablo/right_leg1.STL"
+                       mesh_file="package://diablo_swingarm/description/meshes/diablo/right_leg1.STL"
                        material_name="silver"/>
     <xacro:create_link name="right_leg2" mass="0.18218" ixx="4.1372E-05" ixy="5.1777E-09" ixz="7.3659E-06"
                        iyy="0.00048219" iyz="4.5225E-11" izz="0.00050441"
-                       mesh_file="package://upright_asset/description/meshes/diablo/right_leg2.STL"
+                       mesh_file="package://diablo_swingarm/description/meshes/diablo/right_leg2.STL"
                        material_name="silver"/>
     <xacro:create_link name="right_wheel" mass="2.9494" ixx="0.0069339" ixy="-1.3146E-07" ixz="-3.0392E-09"
                        iyy="0.0069339" iyz="-3.5756E-09" izz="0.012567"
-                       mesh_file="package://upright_asset/description/meshes/diablo/right_wheel.STL"
+                       mesh_file="package://diablo_swingarm/description/meshes/diablo/right_wheel.STL"
                        material_name="black"/>
     <xacro:create_link name="right_leg3" mass="0.071103" ixx="1.6657E-05" ixy="-5.5246E-06" ixz="1.4852E-14"
                        iyy="0.00017966" iyz="-6.5194E-14" izz="0.00019328"
-                       mesh_file="package://upright_asset/description/meshes/diablo/right_leg3.STL"
+                       mesh_file="package://diablo_swingarm/description/meshes/diablo/right_leg3.STL"
                        material_name="brown"/>
     <xacro:create_joint name="left_j4" type="continuous" parent="diablo_base_link" child="left_motor"

File: mobile_manipulator_assets/diablo_swingarm/description/urdf/diablo/robot.xacro (robot description, xacro)
@@ -2,6 +2,6 @@
 <robot xmlns:xacro="http://www.ros.org/wiki/xacro" name="robot">
     <xacro:arg name="robot_type" default="diablo"/>
-    <xacro:include filename="$(find upright_asset)/description/urdf/diablo/diablo.xacro"/>
-    <xacro:include filename="$(find upright_asset)/description/urdf/diablo/gazebo.xacro"/>
-    <!--    <xacro:include filename="$(find upright_asset)/description/urdf/diablo/imu.xacro"/>-->
+    <xacro:include filename="$(find diablo_swingarm)/description/urdf/diablo/diablo.xacro"/>
+    <xacro:include filename="$(find diablo_swingarm)/description/urdf/diablo/gazebo.xacro"/>
+    <!--    <xacro:include filename="$(find diablo_swingarm)/description/urdf/diablo/imu.xacro"/>-->
 </robot>

File: mobile_manipulator_assets/diablo_swingarm/description/urdf/diablo/robot_pinocchio.xacro (robot description, xacro)
@@ -2,50 +2,50 @@
 <robot xmlns:xacro="http://ros.org/wiki/xacro" name="diablo_pinocchio">
     <!-- Include predefined materials -->
-    <xacro:include filename="$(find upright_asset)/description/urdf/common/materials.xacro"/>
-    <xacro:include filename="$(find upright_asset)/description/urdf/common/common.xacro"/>
+        <xacro:include filename="$(find robot_common)/include/robot_common/utilities/urdf/common.xacro"/>
+    <xacro:include filename="$(find robot_common)/include/robot_common/utilities/urdf/materials.xacro"/>
     <!-- Base Link -->
     <xacro:create_link name="diablo_base_link" mass="11.639" ixx="0.071628" ixy="-5.9879E-09" ixz="-0.00097471"
                        iyy="0.16274" iyz="-1.6369E-08" izz="0.14673"
-                       mesh_file="package://upright_asset/description/meshes/diablo/base_link.STL"
+                       mesh_file="package://diablo_swingarm/description/meshes/diablo/base_link.STL"
                        material_name="grey"/>
     <xacro:create_link name="left_motor" mass="1.3837" ixx="0.003352" ixy="2.7785E-09" ixz="-6.5913E-05" iyy="0.0034908"
                        iyz="4.5045E-10" izz="0.0034856"
-                       mesh_file="package://upright_asset/description/meshes/diablo/left_motor.STL"
+                       mesh_file="package://diablo_swingarm/description/meshes/diablo/left_motor.STL"
                        material_name="silver"/>
     <xacro:create_link name="left_leg1" mass="0.10382" ixx="3.6972E-05" ixy="2.4106E-05" ixz="4.3699E-10"
                        iyy="0.00029278" iyz="-4.1243E-11" izz="0.00032532"
-                       mesh_file="package://upright_asset/description/meshes/diablo/left_leg1.STL"
+                       mesh_file="package://diablo_swingarm/description/meshes/diablo/left_leg1.STL"
                        material_name="silver"/>
     <xacro:create_link name="left_leg2" mass="0.18218" ixx="4.1372E-05" ixy="5.1445E-09" ixz="-7.3659E-06"
                        iyy="0.00048219" iyz="2.5521E-11" izz="0.00050441"
-                       mesh_file="package://upright_asset/description/meshes/diablo/left_leg2.STL"
+                       mesh_file="package://diablo_swingarm/description/meshes/diablo/left_leg2.STL"
                        material_name="silver"/>
     <xacro:create_link name="left_wheel" mass="2.9494" ixx="0.0069338" ixy="2.8693E-09" ixz="4.6779E-09" iyy="0.006934"
                        iyz="-5.0441E-11" izz="0.012567"
-                       mesh_file="package://upright_asset/description/meshes/diablo/left_wheel.STL"
+                       mesh_file="package://diablo_swingarm/description/meshes/diablo/left_wheel.STL"
                        material_name="black"/>
     <xacro:create_link name="left_leg3" mass="0.071103" ixx="1.6657E-05" ixy="-5.5246E-06" ixz="3.9598E-14"
                        iyy="0.00017966" iyz="-6.5493E-15" izz="0.00019328"
-                       mesh_file="package://upright_asset/description/meshes/diablo/left_leg3.STL"
+                       mesh_file="package://diablo_swingarm/description/meshes/diablo/left_leg3.STL"
                        material_name="brown"/>
     <xacro:create_link name="right_motor" mass="1.3838" ixx="0.003352" ixy="-2.6527E-09" ixz="6.5914E-05"
                        iyy="0.0034908" iyz="-7.2968E-10" izz="0.0034856"
-                       mesh_file="package://upright_asset/description/meshes/diablo/right_motor.STL"
+                       mesh_file="package://diablo_swingarm/description/meshes/diablo/right_motor.STL"
                        material_name="silver"/>
     <xacro:create_link name="right_leg1" mass="0.10382" ixx="3.6972E-05" ixy="2.4106E-05" ixz="-4.3686E-10"
                        iyy="0.00029278" iyz="4.1459E-11" izz="0.00032532"
-                       mesh_file="package://upright_asset/description/meshes/diablo/right_leg1.STL"
+                       mesh_file="package://diablo_swingarm/description/meshes/diablo/right_leg1.STL"
                        material_name="silver"/>
     <xacro:create_link name="right_leg2" mass="0.18218" ixx="4.1372E-05" ixy="5.1777E-09" ixz="7.3659E-06"
                        iyy="0.00048219" iyz="4.5225E-11" izz="0.00050441"
-                       mesh_file="package://upright_asset/description/meshes/diablo/right_leg2.STL"
+                       mesh_file="package://diablo_swingarm/description/meshes/diablo/right_leg2.STL"
                        material_name="silver"/>
     <xacro:create_link name="right_wheel" mass="2.9494" ixx="0.0069339" ixy="-1.3146E-07" ixz="-3.0392E-09"
                        iyy="0.0069339" iyz="-3.5756E-09" izz="0.012567"
-                       mesh_file="package://upright_asset/description/meshes/diablo/right_wheel.STL"
+                       mesh_file="package://diablo_swingarm/description/meshes/diablo/right_wheel.STL"
                        material_name="black"/>
     <xacro:create_link name="right_leg3" mass="0.071103" ixx="1.6657E-05" ixy="-5.5246E-06" ixz="1.4852E-14"
                        iyy="0.00017966" iyz="-6.5194E-14" izz="0.00019328"
-                       mesh_file="package://upright_asset/description/meshes/diablo/right_leg3.STL"
+                       mesh_file="package://diablo_swingarm/description/meshes/diablo/right_leg3.STL"
                        material_name="brown"/>
     <xacro:create_joint name="left_j4" type="fixed" parent="diablo_base_link" child="left_motor"

File: mobile_manipulator_assets/diablo_swingarm/description/urdf/diablo/transmission.xacro (robot description, xacro)
@@ -1,5 +1,5 @@
 <?xml version="1.0"?>
 <robot xmlns:xacro="http://ros.org/wiki/xacro">
-    <xacro:include filename="$(find upright_asset)/description/urdf/common/common.xacro"/>
+    <xacro:include filename="$(find diablo_swingarm)/description/urdf/common/common.xacro"/>
     <!-- Define transmissions for each joint -->
     <xacro:create_transmission prefix="right" joint_name="j1"/>

File: mobile_manipulator_assets/diablo_swingarm/description/urdf/diablo_manipulator/robot.urdf (robot description, URDF)
Before this commit: robot diablo_rm, 18 links, 17 joints
Links:
- link Link1: geometry collision mesh filename=package://diablo_swingarm/description/meshes/RM65/link1.STL; visual mesh filename=package://diablo_swingarm/description/meshes/RM65/link1.STL
- link Link2: geometry collision mesh filename=package://diablo_swingarm/description/meshes/RM65/link2.STL; visual mesh filename=package://diablo_swingarm/description/meshes/RM65/link2.STL
- link Link3: geometry collision mesh filename=package://diablo_swingarm/description/meshes/RM65/link3.STL; visual mesh filename=package://diablo_swingarm/description/meshes/RM65/link3.STL
- link Link4: geometry collision mesh filename=package://diablo_swingarm/description/meshes/RM65/link4.STL; visual mesh filename=package://diablo_swingarm/description/meshes/RM65/link4.STL
- link Link5: geometry collision mesh filename=package://diablo_swingarm/description/meshes/RM65/link5.STL; visual mesh filename=package://diablo_swingarm/description/meshes/RM65/link5.STL
- link Link6: geometry collision mesh filename=package://diablo_swingarm/description/meshes/RM65/link6.STL; visual mesh filename=package://diablo_swingarm/description/meshes/RM65/link6.STL
- link arm_base_link: geometry collision mesh filename=package://diablo_swingarm/description/meshes/RM65/base_link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; visual mesh filename=package://diablo_swingarm/description/meshes/RM65/base_link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
- link diablo_base_link: geometry collision mesh filename=package://diablo_swingarm/description/meshes/diablo/base_li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 scale=1 1 1; visual mesh filename=package://diablo_swingarm/description/meshes/diablo/base_li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 scale=1 1 1
- link left_leg1: geometry collision mesh filename=package://diablo_swingarm/description/meshes/diablo/left_le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 scale=1 1 1; visual mesh filename=package://diablo_swingarm/description/meshes/diablo/left_le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 scale=1 1 1
- link left_leg2: geometry collision mesh filename=package://diablo_swingarm/description/meshes/diablo/left_le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 scale=1 1 1; visual mesh filename=package://diablo_swingarm/description/meshes/diablo/left_le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 scale=1 1 1
- link left_leg3: geometry collision mesh filename=package://diablo_swingarm/description/meshes/diablo/left_le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 scale=1 1 1; visual mesh filename=package://diablo_swingarm/description/meshes/diablo/left_le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 scale=1 1 1
- link left_motor: geometry collision mesh filename=package://diablo_swingarm/description/meshes/diablo/left_mo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 scale=1 1 1; visual mesh filename=package://diablo_swingarm/description/meshes/diablo/left_mo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 scale=1 1 1
- link left_wheel: geometry collision mesh filename=package://diablo_swingarm/description/meshes/diablo/left_wh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 scale=1 1 1; visual mesh filename=package://diablo_swingarm/description/meshes/diablo/left_wh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 scale=1 1 1
- link right_leg1: geometry collision mesh filename=package://diablo_swingarm/description/meshes/diablo/right_l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 scale=1 1 1; visual mesh filename=package://diablo_swingarm/description/meshes/diablo/right_l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 scale=1 1 1
- link right_leg2: geometry collision mesh filename=package://diablo_swingarm/description/meshes/diablo/right_l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 scale=1 1 1; visual mesh filename=package://diablo_swingarm/description/meshes/diablo/right_l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 scale=1 1 1
- link right_leg3: geometry collision mesh filename=package://diablo_swingarm/description/meshes/diablo/right_l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 scale=1 1 1; visual mesh filename=package://diablo_swingarm/description/meshes/diablo/right_l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 scale=1 1 1
- link right_motor: geometry collision mesh filename=package://diablo_swingarm/description/meshes/diablo/right_m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 scale=1 1 1; visual mesh filename=package://diablo_swingarm/description/meshes/diablo/right_m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 scale=1 1 1
- link right_wheel: geometry collision mesh filename=package://diablo_swingarm/description/meshes/diablo/right_w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 scale=1 1 1; visual mesh filename=package://diablo_swingarm/description/meshes/diablo/right_w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 scale=1 1 1

File: mobile_manipulator_assets/diablo_swingarm/description/urdf/diablo_manipulator/robot.xacro (robot description, xacro)
@@ -2,7 +2,7 @@
 <robot xmlns:xacro="http://www.ros.org/wiki/xacro" name="wlm">
     <xacro:arg name="robot_type" default="ddt"/>
-    <xacro:include filename="$(find upright_asset)/description/urdf/diablo/robot.xacro"/>
+    <xacro:include filename="$(find diablo_swingarm)/description/urdf/diablo/robot.xacro"/>
     <!-- manipulatior -->
-    <xacro:include filename="$(find upright_asset)/description/urdf/manipulator/robot.xacro"/>
+    <xacro:include filename="$(find diablo_swingarm)/description/urdf/manipulator/robot.xacro"/>
     <joint name="manipulator_joint" type="fixed">
         <parent link="diablo_base_link"/>

File: mobile_manipulator_assets/diablo_swingarm/description/urdf/diablo_manipulator/robot_pinocchio.urdf (robot description, URDF)
Before this commit: robot wlm, 18 links, 17 joints
Links:
- link arm_base_link: geometry collision mesh filename=package://diablo_swingarm/description/meshes/manipulator/ba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; visual mesh filename=package://diablo_swingarm/description/meshes/manipulator/ba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
- link diablo_base_link: geometry collision mesh filename=package://diablo_swingarm/description/meshes/diablo/base_li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 scale=1 1 1; visual mesh filename=package://diablo_swingarm/description/meshes/diablo/base_li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 scale=1 1 1
- link left_leg1: geometry collision mesh filename=package://diablo_swingarm/description/meshes/diablo/left_le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 scale=1 1 1; visual mesh filename=package://diablo_swingarm/description/meshes/diablo/left_le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 scale=1 1 1
- link left_leg2: geometry collision mesh filename=package://diablo_swingarm/description/meshes/diablo/left_le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 scale=1 1 1; visual mesh filename=package://diablo_swingarm/description/meshes/diablo/left_le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 scale=1 1 1
- link left_leg3: geometry collision mesh filename=package://diablo_swingarm/description/meshes/diablo/left_le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 scale=1 1 1; visual mesh filename=package://diablo_swingarm/description/meshes/diablo/left_le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 scale=1 1 1
- link left_motor: geometry collision mesh filename=package://diablo_swingarm/description/meshes/diablo/left_mo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 scale=1 1 1; visual mesh filename=package://diablo_swingarm/description/meshes/diablo/left_mo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 scale=1 1 1
- link left_wheel: geometry collision mesh filename=package://diablo_swingarm/description/meshes/diablo/left_wh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 scale=1 1 1; visual mesh filename=package://diablo_swingarm/description/meshes/diablo/left_wh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 scale=1 1 1
- link link1: geometry collision mesh filename=package://diablo_swingarm/description/meshes/manipulator/li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; visual mesh filename=package://diablo_swingarm/description/meshes/manipulator/li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
- link link2: geometry collision mesh filename=package://diablo_swingarm/description/meshes/manipulator/li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; visual mesh filename=package://diablo_swingarm/description/meshes/manipulator/li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
- link link3: geometry collision mesh filename=package://diablo_swingarm/description/meshes/manipulator/li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; visual mesh filename=package://diablo_swingarm/description/meshes/manipulator/li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
- link link4: geometry collision mesh filename=package://diablo_swingarm/description/meshes/manipulator/li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; visual mesh filename=package://diablo_swingarm/description/meshes/manipulator/li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
- link link5: geometry collision mesh filename=package://diablo_swingarm/description/meshes/manipulator/li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; visual mesh filename=package://diablo_swingarm/description/meshes/manipulator/li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
- link link6: geometry collision mesh filename=package://diablo_swingarm/description/meshes/manipulator/li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; visual mesh filename=package://diablo_swingarm/description/meshes/manipulator/li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
- link right_leg1: geometry collision mesh filename=package://diablo_swingarm/description/meshes/diablo/right_l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 scale=1 1 1; visual mesh filename=package://diablo_swingarm/description/meshes/diablo/right_l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 scale=1 1 1
- link right_leg2: geometry collision mesh filename=package://diablo_swingarm/description/meshes/diablo/right_l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 scale=1 1 1; visual mesh filename=package://diablo_swingarm/description/meshes/diablo/right_l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 scale=1 1 1
- link right_leg3: geometry collision mesh filename=package://diablo_swingarm/description/meshes/diablo/right_l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 scale=1 1 1; visual mesh filename=package://diablo_swingarm/description/meshes/diablo/right_l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 scale=1 1 1
- link right_motor: geometry collision mesh filename=package://diablo_swingarm/description/meshes/diablo/right_m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 scale=1 1 1; visual mesh filename=package://diablo_swingarm/description/meshes/diablo/right_m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 scale=1 1 1
- link right_wheel: geometry collision mesh filename=package://diablo_swingarm/description/meshes/diablo/right_w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 scale=1 1 1; visual mesh filename=package://diablo_swingarm/description/meshes/diablo/right_w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 scale=1 1 1

File: mobile_manipulator_assets/diablo_swingarm/description/urdf/diablo_manipulator/robot_pinocchio.xacro (robot description, xacro)
@@ -2,7 +2,7 @@
 <robot xmlns:xacro="http://www.ros.org/wiki/xacro" name="wlm">
     <xacro:arg name="robot_type" default="ddt"/>
-    <xacro:include filename="$(find upright_asset)/description/urdf/diablo/robot_pinocchio.xacro"/>
+    <xacro:include filename="$(find diablo_swingarm)/description/urdf/diablo/robot_pinocchio.xacro"/>
     <!-- manipulatior -->
-    <xacro:include filename="$(find upright_asset)/description/urdf/manipulator/robot.xacro"/>
+    <xacro:include filename="$(find diablo_swingarm)/description/urdf/manipulator/robot.xacro"/>
     <joint name="manipulator_joint" type="fixed">
         <parent link="diablo_base_link"/>
