Commit message: Change urdf package.

File: mobile_manipulator_assets/diablo_swingarm/description/urdf/diablo_manipulator/robot_webots.urdf (robot description, URDF)
Before this commit: robot diablo_manipulator, 18 links, 17 joints
Links:
- link arm_base_link: geometry collision mesh filename=package://diablo_swingarm/description/meshes/manipulator/ba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; visual mesh filename=package://diablo_swingarm/description/meshes/manipulator/ba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
- link diablo_base_link: geometry collision mesh filename=package://diablo_swingarm/description/meshes/diablo/base_li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; visual mesh filename=package://diablo_swingarm/description/meshes/diablo/base_li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
- link left_leg1: geometry collision mesh filename=package://diablo_swingarm/description/meshes/diablo/left_le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; visual mesh filename=package://diablo_swingarm/description/meshes/diablo/left_le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
- link left_leg2: geometry collision mesh filename=package://diablo_swingarm/description/meshes/diablo/left_le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; visual mesh filename=package://diablo_swingarm/description/meshes/diablo/left_le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
- link left_leg3: geometry collision mesh filename=package://diablo_swingarm/description/meshes/diablo/left_le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; visual mesh filename=package://diablo_swingarm/description/meshes/diablo/left_le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
- link left_motor: geometry collision mesh filename=package://diablo_swingarm/description/meshes/diablo/left_mo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; visual mesh filename=package://diablo_swingarm/description/meshes/diablo/left_mo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
- link left_wheel: geometry collision mesh filename=package://diablo_swingarm/description/meshes/diablo/left_wh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; visual mesh filename=package://diablo_swingarm/description/meshes/diablo/left_wh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
- link link1: geometry collision mesh filename=package://diablo_swingarm/description/meshes/manipulator/li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; visual mesh filename=package://diablo_swingarm/description/meshes/manipulator/li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
- link link2: geometry collision mesh filename=package://diablo_swingarm/description/meshes/manipulator/li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; visual mesh filename=package://diablo_swingarm/description/meshes/manipulator/li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
- link link3: geometry collision mesh filename=package://diablo_swingarm/description/meshes/manipulator/li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; visual mesh filename=package://diablo_swingarm/description/meshes/manipulator/li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
- link link4: geometry collision mesh filename=package://diablo_swingarm/description/meshes/manipulator/li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; visual mesh filename=package://diablo_swingarm/description/meshes/manipulator/li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
- link link5: geometry collision mesh filename=package://diablo_swingarm/description/meshes/manipulator/li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; visual mesh filename=package://diablo_swingarm/description/meshes/manipulator/li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
- link link6: geometry collision mesh filename=package://diablo_swingarm/description/meshes/manipulator/li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; visual mesh filename=package://diablo_swingarm/description/meshes/manipulator/li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
- link right_leg1: geometry collision mesh filename=package://diablo_swingarm/description/meshes/diablo/right_l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; visual mesh filename=package://diablo_swingarm/description/meshes/diablo/right_l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
- link right_leg2: geometry collision mesh filename=package://diablo_swingarm/description/meshes/diablo/right_l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; visual mesh filename=package://diablo_swingarm/description/meshes/diablo/right_l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
- link right_leg3: geometry collision mesh filename=package://diablo_swingarm/description/meshes/diablo/right_l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; visual mesh filename=package://diablo_swingarm/description/meshes/diablo/right_l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
- link right_motor: geometry collision mesh filename=package://diablo_swingarm/description/meshes/diablo/right_m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; visual mesh filename=package://diablo_swingarm/description/meshes/diablo/right_m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
- link right_wheel: geometry collision mesh filename=package://diablo_swingarm/description/meshes/diablo/right_w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; visual mesh filename=package://diablo_swingarm/description/meshes/diablo/right_w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

File: mobile_manipulator_assets/diablo_swingarm/description/urdf/manipulator/arm.urdf.xacro (robot description, xacro)
@@ -1,10 +1,10 @@
 <?xml version="1.0"?>
 <robot xmlns:xacro="http://ros.org/wiki/xacro" name="arm">
-    <xacro:include filename="$(find upright_asset)/description/urdf/manipulator/common.xacro"/>
-    <!--    <xacro:include filename="$(find upright_asset)/description/urdf/common/materials.xacro"/>-->
+    <xacro:include filename="$(find diablo_swingarm)/description/urdf/manipulator/common.xacro"/>
+    <!--    <xacro:include filename="$(find diablo_swingarm)/description/urdf/common/materials.xacro"/>-->
     <xacro:create_link name="arm_base_link" mass="6.722526"
                        ixx="49640000" ixy="-6571.312" ixz="-906.394"
                        iyy="38820000" iyz="211.811" izz="83030000"
-                       mesh_file="package://upright_asset/description/meshes/manipulator/base_link.stl"
+                       mesh_file="package://diablo_swingarm/description/meshes/manipulator/base_link.stl"
                        material_name="silver"
                        inertial_xyz="0.00006 -0.000046 0.0129"/>
@@ -12,5 +12,5 @@
                        ixx="572600" ixy="-54.105" ixz="-3.821"
                        iyy="495300" iyz="12915.759" izz="538300"
-                       mesh_file="package://upright_asset/description/meshes/manipulator/link1.stl"
+                       mesh_file="package://diablo_swingarm/description/meshes/manipulator/link1.stl"
                        material_name="silver"
                        inertial_xyz="0.000002 -0.00531 0.034685"/>
@@ -18,5 +18,5 @@
                        ixx="383700" ixy="-26179.433" ixz="693.218"
                        iyy="1888000" iyz="-585.018" izz="2050000"
-                       mesh_file="package://upright_asset/description/meshes/manipulator/link2.stl"
+                       mesh_file="package://diablo_swingarm/description/meshes/manipulator/link2.stl"
                        material_name="silver"
                        inertial_xyz="-0.197351 -0.002165 0.000057"/>
@@ -24,5 +24,5 @@
                        ixx="1204000" ixy="-51994.358" ixz="-2550000"
                        iyy="11300000" iyz="-16633.832" izz="10760000"
-                       mesh_file="package://upright_asset/description/meshes/manipulator/link3.stl"
+                       mesh_file="package://diablo_swingarm/description/meshes/manipulator/link3.stl"
                        material_name="silver"
                        inertial_xyz="0.100486 -0.002073 0.028338"/>
@@ -30,5 +30,5 @@
                        ixx="1262.246" ixy="32.61" ixz="-553.334"
                        iyy="1346.829" iyz="41.18" izz="975.984"
-                       mesh_file="package://upright_asset/description/meshes/manipulator/link4.stl"
+                       mesh_file="package://diablo_swingarm/description/meshes/manipulator/link4.stl"
                        material_name="silver"
                        inertial_xyz="0.02969 0.00192 0.03765"/>
@@ -36,9 +36,9 @@
                        ixx="735400" ixy="-449.048" ixz="37386.443"
                        iyy="732800" iyz="-210.043" izz="238600"
-                       mesh_file="package://upright_asset/description/meshes/manipulator/link5.stl"
+                       mesh_file="package://diablo_swingarm/description/meshes/manipulator/link5.stl"
                        material_name="silver"
                        inertial_xyz="0.001992 -0.000088 -0.053421"/>
     <xacro:create_link name="link6" mass="0.001" ixx="10.630412" ixy="-1.068E-10" ixz="83.57" iyy="8414.108" iyz="0.00"
-                       izz="6931.832" mesh_file="package://upright_asset/description/meshes/manipulator/link6.stl"
+                       izz="6931.832" mesh_file="package://diablo_swingarm/description/meshes/manipulator/link6.stl"
                        material_name="silver"/>
     <!-- Joint definitions -->

File: mobile_manipulator_assets/diablo_swingarm/description/urdf/manipulator/gazebo.xacro (robot description, xacro)
@@ -1,5 +1,5 @@
 <?xml version="1.0"?>
 <robot xmlns:xacro="http://ros.org/wiki/xacro" name="gazebo">
-    <xacro:include filename="$(find upright_asset)/description/urdf/manipulator/common.xacro"/>
+    <xacro:include filename="$(find diablo_swingarm)/description/urdf/manipulator/common.xacro"/>
     <!-- Transmission definitions -->
     <xacro:create_transmission joint_name="joint1"/>

File: mobile_manipulator_assets/diablo_swingarm/description/urdf/manipulator/robot.urdf (robot description, URDF)
Before this commit: robot swingboy_v1, 7 links, 6 joints
Links:
- link arm_base_link: geometry collision mesh filename=package://diablo_swingarm/description/meshes/manipulator/ba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; visual mesh filename=package://diablo_swingarm/description/meshes/manipulator/ba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
- link link1: geometry collision mesh filename=package://diablo_swingarm/description/meshes/manipulator/li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; visual mesh filename=package://diablo_swingarm/description/meshes/manipulator/li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
- link link2: geometry collision mesh filename=package://diablo_swingarm/description/meshes/manipulator/li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; visual mesh filename=package://diablo_swingarm/description/meshes/manipulator/li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
- link link3: geometry collision mesh filename=package://diablo_swingarm/description/meshes/manipulator/li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; visual mesh filename=package://diablo_swingarm/description/meshes/manipulator/li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
- link link4: geometry collision mesh filename=package://diablo_swingarm/description/meshes/manipulator/li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; visual mesh filename=package://diablo_swingarm/description/meshes/manipulator/li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
- link link5: geometry collision mesh filename=package://diablo_swingarm/description/meshes/manipulator/li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; visual mesh filename=package://diablo_swingarm/description/meshes/manipulator/li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
- link link6: geometry collision mesh filename=package://diablo_swingarm/description/meshes/manipulator/li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; visual mesh filename=package://diablo_swingarm/description/meshes/manipulator/li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

File: mobile_manipulator_assets/diablo_swingarm/description/urdf/manipulator/robot.xacro (robot description, xacro)
@@ -1,5 +1,5 @@
 <?xml version="1.0"?>
 <robot xmlns:xacro="http://ros.org/wiki/xacro" name="swingboy_v1">
-    <xacro:include filename="$(find upright_asset)/description/urdf/manipulator/arm.urdf.xacro"/>
-    <xacro:include filename="$(find upright_asset)/description/urdf/manipulator/gazebo.xacro"/>
+    <xacro:include filename="$(find diablo_swingarm)/description/urdf/manipulator/arm.urdf.xacro"/>
+    <xacro:include filename="$(find diablo_swingarm)/description/urdf/manipulator/gazebo.xacro"/>
 </robot>
