Commit message: Build right but very strange problem.

File: mobile_manipulator_assets/diablo/description/urdf/diablo.urdf.xacro (robot description, xacro)
@@ -2,73 +2,95 @@
 <robot xmlns:xacro="http://ros.org/wiki/xacro">
     <!-- Include predefined materials -->
+    <xacro:include filename="$(find robot_common)/include/robot_common/utilities/urdf/imu.urdf.xacro"/>
     <xacro:include filename="$(find robot_common)/include/robot_common/utilities/urdf/common.xacro"/>
-    <xacro:include filename="$(find robot_common)/include/robot_common/utilities/urdf/materials.xacro"/>
-    <xacro:include filename="$(find robot_common)/include/robot_common/utilities/urdf/imu.urdf.xacro"/>
     <!-- Base Link -->
-<!--    <link name="world"/>-->
-    <xacro:create_link name="diablo_base_link" mass="11.639" ixx="0.071628" ixy="-5.9879E-09" ixz="-0.00097471"
-                       iyy="0.16274" iyz="-1.6369E-08" izz="0.14673"
-                       mesh_file="package://diablo/description/meshes/base_link.stl"
-                       material_name="grey" scale_factor="1" vision_scale_x="0.1" vision_scale_y="0.1" vision_scale_z="0.1"
-                       collision_scale_x="0.1" collision_scale_y="0.001" collision_scale_z="0.1"/>
-    <xacro:IMU connected_to="diablo_base_link" imu_name="base_imu" mesh_file="package://robot_common/include/robot_common/utilities/urdf/imu.stl" xyz="0.00 0.00 0.00"
+    <link name="diablo_base_link">
+        <inertial>
+            <origin xyz="0 0 0" rpy="0 0 0"/>
+            <mass value="11.639"/>
+            <inertia ixx="0.071628" ixy="-5.9879E-09" ixz="-0.00097471"
+                     iyy="0.16274" iyz="-1.6369E-08" izz="0.14673"/>
+        </inertial>
+        <visual>
+            <origin xyz="0 0 0" rpy="0 0 0"/>
+            <geometry>
+                <mesh filename="package://diablo/description/meshes/base_link.stl"
+                      scale="0.10 0.10 0.10"/>
+            </geometry>
+        </visual>
+        <collision>
+            <origin xyz="0 0 0" rpy="0 0 0"/>
+            <geometry>
+                <mesh filename="package://diablo/description/meshes/base_link.stl"
+                      scale="0.10 0.010 0.10"/>
+            </geometry>
+        </collision>
+    </link>
+    <xacro:IMU connected_to="diablo_base_link" imu_name="base_imu"
+               mesh_file="package://robot_common/include/robot_common/utilities/urdf/imu.stl" xyz="0.00 0.00 0.00"
                rpy="0.00 0.00 0.00"/>
     <xacro:create_link name="left_motor" mass="1.3837" ixx="0.003352" ixy="2.7785E-09" ixz="-6.5913E-05" iyy="0.0034908"
                        iyz="4.5045E-10" izz="0.0034856"
                        mesh_file="package://diablo/description/meshes/left_motor.STL"
-                       material_name="silver" scale_factor="1"/>
+                       scale_factor="1"/>
     <xacro:create_link name="left_leg1" mass="0.10382" ixx="3.6972E-05" ixy="2.4106E-05" ixz="4.3699E-10"
                        iyy="0.00029278" iyz="-4.1243E-11" izz="0.00032532"
                        mesh_file="package://diablo/description/meshes/left_leg1.STL"
-                       material_name="silver" scale_factor="1"/>
+                       scale_factor="1"/>
     <xacro:create_link name="left_leg2" mass="0.18218" ixx="4.1372E-05" ixy="5.1445E-09" ixz="-7.3659E-06"
                        iyy="0.00048219" iyz="2.5521E-11" izz="0.00050441"
                        mesh_file="package://diablo/description/meshes/left_leg2.STL"
-                       material_name="silver" scale_factor="1"/>
+                       scale_factor="1"/>
     <xacro:create_link name="left_wheel" mass="2.9494" ixx="0.0069338" ixy="2.8693E-09" ixz="4.6779E-09" iyy="0.006934"
                        iyz="-5.0441E-11" izz="0.012567"
                        mesh_file="package://diablo/description/meshes/left_wheel.STL"
-                       material_name="black" scale_factor="1"/>
+                       scale_factor="1"/>
     <xacro:create_link name="left_leg3" mass="0.071103" ixx="1.6657E-05" ixy="-5.5246E-06" ixz="3.9598E-14"
                        iyy="0.00017966" iyz="-6.5493E-15" izz="0.00019328"
                        mesh_file="package://diablo/description/meshes/left_leg3.STL"
-                       material_name="brown" scale_factor="1"/>
+                       scale_factor="1"/>
     <xacro:create_link name="right_motor" mass="1.3838" ixx="0.003352" ixy="-2.6527E-09" ixz="6.5914E-05"
                        iyy="0.0034908" iyz="-7.2968E-10" izz="0.0034856"
                        mesh_file="package://diablo/description/meshes/right_motor.STL"
-                       material_name="silver" scale_factor="1"/>
+                       scale_factor="1"/>
     <xacro:create_link name="right_leg1" mass="0.10382" ixx="3.6972E-05" ixy="2.4106E-05" ixz="-4.3686E-10"
                        iyy="0.00029278" iyz="4.1459E-11" izz="0.00032532"
                        mesh_file="package://diablo/description/meshes/right_leg1.STL"
-                       material_name="silver" scale_factor="1"/>
+                       scale_factor="1"/>
     <xacro:create_link name="right_leg2" mass="0.18218" ixx="4.1372E-05" ixy="5.1777E-09" ixz="7.3659E-06"
                        iyy="0.00048219" iyz="4.5225E-11" izz="0.00050441"
                        mesh_file="package://diablo/description/meshes/right_leg2.STL"
-                       material_name="silver" scale_factor="1"/>
+                       scale_factor="1"/>
     <xacro:create_link name="right_wheel" mass="2.9494" ixx="0.0069339" ixy="-1.3146E-07" ixz="-3.0392E-09"
                        iyy="0.0069339" iyz="-3.5756E-09" izz="0.012567"
                        mesh_file="package://diablo/description/meshes/right_wheel.STL"
-                       material_name="black" scale_factor="1"/>
+                       scale_factor="1"/>
     <xacro:create_link name="right_leg3" mass="0.071103" ixx="1.6657E-05" ixy="-5.5246E-06" ixz="1.4852E-14"
                        iyy="0.00017966" iyz="-6.5194E-14" izz="0.00019328"
                        mesh_file="package://diablo/description/meshes/right_leg3.STL"
-                       material_name="brown" scale_factor="1"/>
+                       scale_factor="1"/>
     <xacro:macro name="chassis" params="fixed_wheel fixed_leg='false'">
         <xacro:unless value="${fixed_leg}">
             <xacro:create_joint name="left_j4" type="continuous" parent="diablo_base_link" child="left_motor"
                                 origin_xyz="0 0.18755 0" origin_rpy="1.5708 0.13433 -3.1416" axis_xyz="0 0 1"/>
-            <xacro:create_joint name="left_j1" type="continuous" parent="left_motor" child="left_leg1" origin_xyz="0 0 0"
+            <xacro:create_joint name="left_j1" type="continuous" parent="left_motor" child="left_leg1"
+                                origin_xyz="0 0 0"
                                 origin_rpy="0 0 -2.8729" axis_xyz="0 0 1"/>
-            <xacro:create_joint name="left_j2" type="continuous" parent="left_leg1" child="left_leg2" origin_xyz="0.14 0 0"
+            <xacro:create_joint name="left_j2" type="continuous" parent="left_leg1" child="left_leg2"
+                                origin_xyz="0.14 0 0"
                                 origin_rpy="0 0 2.8729" axis_xyz="0 0 1"/>
-            <xacro:create_joint name="left_j5" type="continuous" parent="left_motor" child="left_leg3" origin_xyz="0.09 0 0"
+            <xacro:create_joint name="left_j5" type="continuous" parent="left_motor" child="left_leg3"
+                                origin_xyz="0.09 0 0"
                                 origin_rpy="0 0 -2.8729" axis_xyz="0 0 1"/>
             <xacro:create_joint name="right_j4" type="continuous" parent="diablo_base_link" child="right_motor"
                                 origin_xyz="0 -0.18755 0" origin_rpy="1.5708 0.13433 3.1416" axis_xyz="0 0 1"/>
-            <xacro:create_joint name="right_j1" type="continuous" parent="right_motor" child="right_leg1" origin_xyz="0 0 0"
+            <xacro:create_joint name="right_j1" type="continuous" parent="right_motor" child="right_leg1"
+                                origin_xyz="0 0 0"
                                 origin_rpy="0 0 -2.8729" axis_xyz="0 0 1"/>
-            <xacro:create_joint name="right_j2" type="continuous" parent="right_leg1" child="right_leg2" origin_xyz="0.14 0 0"
+            <xacro:create_joint name="right_j2" type="continuous" parent="right_leg1" child="right_leg2"
+                                origin_xyz="0.14 0 0"
                                 origin_rpy="0 0 2.8729" axis_xyz="0 0 1"/>
-            <xacro:create_joint name="right_j5" type="continuous" parent="right_motor" child="right_leg3" origin_xyz="0.09 0 0"
+            <xacro:create_joint name="right_j5" type="continuous" parent="right_motor" child="right_leg3"
+                                origin_xyz="0.09 0 0"
                                 origin_rpy="0 0 -2.8729" axis_xyz="0 0 1"/>
             <!-- Define transmissions for each joint -->
@@ -95,7 +117,9 @@
             <xacro:create_joint name="right_j1" type="fixed" parent="right_motor" child="right_leg1" origin_xyz="0 0 0"
                                 origin_rpy="0 0 -2.8729" axis_xyz="0 0 1"/>
-            <xacro:create_joint name="right_j2" type="fixed" parent="right_leg1" child="right_leg2" origin_xyz="0.14 0 0"
+            <xacro:create_joint name="right_j2" type="fixed" parent="right_leg1" child="right_leg2"
+                                origin_xyz="0.14 0 0"
                                 origin_rpy="0 0 2.8729" axis_xyz="0 0 1"/>
-            <xacro:create_joint name="right_j5" type="fixed" parent="right_motor" child="right_leg3" origin_xyz="0.09 0 0"
+            <xacro:create_joint name="right_j5" type="fixed" parent="right_motor" child="right_leg3"
+                                origin_xyz="0.09 0 0"
                                 origin_rpy="0 0 -2.8729" axis_xyz="0 0 1"/>
         </xacro:if>
@@ -145,34 +169,9 @@
         <self_collide>1</self_collide>
     </gazebo>
-    <gazebo reference="left_wheel">
-        <material>Gazebo/Purple</material>
-    </gazebo>
-    <gazebo reference="right_wheel">
-        <material>Gazebo/Purple</material>
-    </gazebo>
-    <gazebo reference="diablo_base_link">
-        <material>
-            <friction>
-                <ode>
-                    <mu>0.0</mu>  <!-- 设置mu1为0 -->
-                    <mu2>0.0</mu2>  <!-- 设置mu2为0 -->
-                </ode>
-            </friction>
-        </material>
-        <self_collide>false</self_collide>  <!-- 设置为false -->
-        <kp>1000000.0</kp>  <!-- 接触刚度参数 -->
-        <kd>10.0</kd>  <!-- 接触阻尼参数 -->
-    </gazebo>
-    <!--    <gazebo reference="diablo_base_link">-->
-<!--        <mu1>0.</mu1>-->
-<!--        <mu2>0.</mu2>-->
-<!--        <self_collide>0</self_collide>-->
-<!--        <kp value="1000000.0"/>-->
-<!--        <kd value="10.0"/>-->
+<!--    <gazebo reference="left_wheel">-->
+<!--        <material>Gazebo/Purple</material>-->
 <!--    </gazebo>-->
-<!--    <gazebo>-->
-<!--        <plugin name="gazebo_ros_control" filename="libgazebo_ros_control.so">-->
-<!--            <robotNamespace>/</robotNamespace>-->
-<!--        </plugin>-->
+<!--    <gazebo reference="right_wheel">-->
+<!--        <material>Gazebo/Purple</material>-->
 <!--    </gazebo>-->
 </robot>

File: mobile_manipulator_assets/diablo/description/urdf/robot.xacro (robot description, xacro)
@@ -3,6 +3,6 @@
     <xacro:arg name="robot_type" default="diablo"/>
     <xacro:arg name="load_chassis" default="true"/>
-    <xacro:arg name="fixed_leg" default="false"/>
-    <xacro:arg name="fixed_wheel" default="true"/>
+    <xacro:arg name="fixed_leg" default="true"/>
+    <xacro:arg name="fixed_wheel" default="false"/>
     <xacro:if value="$(arg load_chassis)">
         <xacro:include filename="$(find diablo)/description/urdf/diablo.urdf.xacro"/>

File: mobile_manipulator_assets/diablo_swingarm/description/urdf/gazebo_robot.xacro (robot description, xacro)
@@ -1,12 +1,6 @@
 <?xml version="1.0"?>
 <robot xmlns:xacro="http://www.ros.org/wiki/xacro" name="wlm">
-    <xacro:arg name="robot_type" default="ddt"/>
     <!-- manipulatior -->
     <xacro:include filename="$(find swing_arm)/description/urdf/robot.xacro"/>
-    <joint name="manipulator_joint" type="fixed">
-        <parent link="diablo_base_link"/>
-        <child link="arm_base_link"/>
-        <origin xyz="0.0 0.0 0.1" rpy="0.0 0.0 0.0"/>
-    </joint>
     <xacro:arg name="load_chassis" default="true"/>
     <xacro:arg name="fixed_leg" default="true"/>
@@ -16,10 +10,9 @@
         <xacro:chassis fixed_wheel="$(arg fixed_wheel)" fixed_leg="$(arg fixed_leg)"/>
     </xacro:if>
-<!--    <gazebo>-->
-<!--        <plugin name="gazebo_ros_control" filename="libgazebo_ros_control.so">-->
-<!--            <robotNamespace>/</robotNamespace>-->
-<!--            <robotParam>mobile_manipulator_description</robotParam>-->
-<!--        </plugin>-->
-<!--    </gazebo>-->
+    <joint name="manipulator_joint" type="fixed">
+        <parent link="diablo_base_link"/>
+        <child link="arm_base_link"/>
+        <origin xyz="0.0 0.0 0.1" rpy="0.0 0.0 0.0"/>
+    </joint>
     <gazebo>
         <plugin name="gazebo_ros_control" filename="libmobile_manipulator_hw_sim.so">

File: mobile_manipulator_assets/swing_arm/description/urdf/arm.urdf.xacro (robot description, xacro)
@@ -2,24 +2,23 @@
 <robot xmlns:xacro="http://ros.org/wiki/xacro" name="swingarm">
     <xacro:include filename="$(find robot_common)/include/robot_common/utilities/urdf/common.xacro"/>
-    <xacro:include filename="$(find robot_common)/include/robot_common/utilities/urdf/materials.xacro"/>
     <xacro:create_link name="arm_base_link" mass="6.722526"
                        ixx="49640000" ixy="-6571.312" ixz="-906.394"
                        iyy="38820000" iyz="211.811" izz="83030000"
-                       mesh_file="package://swing_arm/description/meshes/base_link.stl" material_name="silver"
+                       mesh_file="package://swing_arm/description/meshes/baselink.stl"
                        inertial_xyz="0.00006 -0.000046 0.0129"/>
     <xacro:create_link name="link1" mass="1.103721"
                        ixx="572600" ixy="-54.105" ixz="-3.821"
                        iyy="495300" iyz="12915.759" izz="538300"
-                       mesh_file="package://swing_arm/description/meshes/link1.stl" material_name="silver"
+                       mesh_file="package://swing_arm/description/meshes/link1.stl"
                        inertial_xyz="0.000002 -0.00531 0.034685"/>
     <xacro:create_link name="link2" mass="0.734276"
                        ixx="383700" ixy="-26179.433" ixz="693.218"
                        iyy="1888000" iyz="-585.018" izz="2050000"
-                       mesh_file="package://swing_arm/description/meshes/link2.stl" material_name="silver"
+                       mesh_file="package://swing_arm/description/meshes/link2.stl"
                        inertial_xyz="-0.197351 -0.002165 0.000057"/>
     <xacro:create_link name="link3" mass="0.474451"
                        ixx="322900" ixy="8650.968" ixz="-231700"
                        iyy="2226000" iyz="1036.356" izz="2291000"
-                       mesh_file="package://swing_arm/description/meshes/link3.stl" material_name="silver"
+                       mesh_file="package://swing_arm/description/meshes/link3.stl"
                        inertial_xyz="0.191296 -0.001405 0.053882"
                        collision_scale_y="0.8"/>
@@ -27,12 +26,12 @@
                        ixx="1262.246" ixy="32.61" ixz="-553.334"
                        iyy="100000" iyz="41.18" izz="975.984"
-                       mesh_file="package://swing_arm/description/meshes/link4.stl" material_name="silver"
+                       mesh_file="package://swing_arm/description/meshes/link4.stl"
                        inertial_xyz="0.02969 0.00192 0.03765"/>
     <xacro:create_link name="link5" mass="0.598593"
                        ixx="735400" ixy="-449.048" ixz="37386.443"
                        iyy="732800" iyz="-210.043" izz="500000"
-                       mesh_file="package://swing_arm/description/meshes/link5.stl" material_name="silver"
+                       mesh_file="package://swing_arm/description/meshes/link5.stl"
                        inertial_xyz="0.001992 -0.000088 -0.053421"/>
-    <xacro:create_link name="link6" mass="0.5" ixx="50000" ixy="-1.068E-10" ixz="83.57" iyy="8414.108" iyz="0.00" izz="6931.832" mesh_file="package://swing_arm/description/meshes/link6.stl" material_name="silver"/>
+    <xacro:create_link name="link6" mass="0.5" ixx="50000" ixy="-1.068E-10" ixz="83.57" iyy="8414.108" iyz="0.00" izz="6931.832" mesh_file="package://swing_arm/description/meshes/link6.stl" />
     <!-- Joint definitions -->
     <xacro:create_joint name="joint1" type="revolute" parent="arm_base_link" child="link1" origin_xyz="0 0 0.07925" origin_rpy="0 0 0" axis_xyz="0 0 1" lower="-1.57" upper="1.57" effort="30" velocity="1.5"/>
